Commit message: smaller urdf

File: urdf/ceres_velodyne.urdf.xacro (robot description, xacro)
@@ -5,293 +5,267 @@
   xmlns:interface="http://playerstage.sourceforge.net/gazebo/xmlschema/#interface"
   xmlns:sensor="http://playerstage.sourceforge.net/gazebo/xmlschema/#sensor"
-  name="ceres">
-  <xacro:include filename="$(find uos_common_urdf)/common.xacro" />
-  <xacro:include filename="$(find uos_common_urdf)/urdf/imu.gazebo.urdf.xacro" />
-  <xacro:property name="M_PI" value="3.14159265359"/>
-  <xacro:property name="imu_stdev" value="0.00017" />
-  <xacro:property name="body_height" value="0.15"/>
-  <xacro:property name="body_length" value="0.38"/>
-  <xacro:property name="body_width" value="0.32"/>
-  <xacro:property name="axis_front" value="0.14"/>
-  <xacro:property name="axis_back" value="-0.14"/>
-  <xacro:property name="wheel_thickness" value="0.085"/>
-  <xacro:property name="wheel_body_offset" value="${wheel_thickness/2 + 0.015}"/>
-  <xacro:property name="wheel_radius" value="0.135"/>
-  <xacro:property name="axis_height" value="-0.03"/>
-  <xacro:property name="axis_right" value="${-body_width/2 - wheel_body_offset}"/>
-  <xacro:property name="axis_left" value="${body_width/2 + wheel_body_offset}"/>
-  <xacro:property name="axis_length" value="${body_width + 2 * wheel_body_offset}" />
-  <xacro:property name="turning_adaptation" value="0.95" />
-  <xacro:property name="bearing_width" value="0.05"/>
-  <xacro:property name="bearing_height" value="0.09"/>
-  <xacro:property name="bearing_thickness" value="0.01"/>
-  <xacro:property name="body_mass" value="40.0"/>
-  <xacro:property name="wheel_mass" value="3.0"/>
-  <xacro:property name="imu_width" value="0.036"/>
-  <xacro:property name="imu_length" value="0.038"/>
-  <xacro:property name="imu_height" value="0.012"/>
-  <xacro:property name="imu_offset_x" value="0"/>
-  <xacro:property name="imu_offset_y" value="0"/>
-  <xacro:property name="imu_offset_z" value="${- body_height/2 + 0.005 + 0.007}"/>
-  <xacro:property name="em_body_length" value="0.11"/>
-  <xacro:property name="em_body_width" value="0.04"/>
-  <xacro:property name="em_body_height" value="0.03"/>
-  <xacro:property name="em_button_radius" value="0.0125"/>
-  <xacro:property name="em_button_depth" value="0.02" />
-  <xacro:property name="velodyne_height" value="0.1442"/>
-  <xacro:property name="velodyne_radius" value="0.04265"/>
-  <xacro:property name="velodyne_height_to_lense" value="0.090805"/>
-  <!--<xacro:property name="velodyne_offset_x" value="${body_length/2 - 0.0265 + 0.02}"/>
-  <xacro:property name="velodyne_offset_y" value="0"/>
-  <xacro:property name="velodyne_offset_z"
-    value="${-0.005 + velodyne_height/2}"/> -->
-  <xacro:property name="velodyne_offset_x" value="${body_length/2 - 0.0265 + 0.02}"/>
-  <xacro:property name="velodyne_offset_y" value="0"/>
-  <xacro:property name="velodyne_offset_z"
-    value="${0.2 + velodyne_height/2}"/>
-  <link name="base_footprint"/>
-  <link name="base_link">
-    <visual>
-      <origin xyz="0 0 0" rpy="0 0 0" />
+  name="robot">
+<xacro:macro name="box_inertial" params="x y z mass">
+    <inertial>
+    <mass value="${mass}" />
+    <origin xyz="0 0 0" />
+    <inertia ixx="${0.0833333 * mass * (y*y + z*z)}" ixy="0.0" ixz="0.0"
+        iyy="${0.0833333 * mass * (x*x + z*z)}" iyz="0.0"
+        izz="${0.0833333 * mass * (x*x + y*y)}" />
+    </inertial>
+</xacro:macro>
+<xacro:macro name="cylinder_inertial_with_origin" params="radius length mass *origin">
+<inertial>
+    <mass value="${mass}" />
+    <xacro:insert_block name="origin" />
+    <inertia ixx="${0.0833333 * mass * (3 * radius * radius + length * length)}" ixy="0.0" ixz="0.0"
+    iyy="${0.0833333 * mass * (3 * radius * radius + length * length)}" iyz="0.0"
+    izz="${0.5 * mass * radius * radius}" />
+</inertial>
+</xacro:macro>
+<xacro:property name="M_PI" value="3.14159265359"/>
+<xacro:property name="imu_stdev" value="0.00017" />
+<xacro:property name="body_height" value="0.15"/>
+<xacro:property name="body_length" value="0.38"/>
+<xacro:property name="body_width" value="0.32"/>
+<xacro:property name="axis_front" value="0.14"/>
+<xacro:property name="axis_back" value="-0.14"/>
+<xacro:property name="wheel_thickness" value="0.07"/>
+<xacro:property name="wheel_body_offset" value="${wheel_thickness/2 + 0.015}"/>
+<xacro:property name="wheel_radius" value="0.135"/>
+<xacro:property name="axis_height" value="-0.03"/>
+<xacro:property name="axis_right" value="${-body_width/2 - wheel_body_offset}"/>
+<xacro:property name="axis_left" value="${body_width/2 + wheel_body_offset}"/>
+<xacro:property name="axis_length" value="${body_width + 2 * wheel_body_offset}" />
+<xacro:property name="turning_adaptation" value="2.95" />
+<xacro:property name="body_mass" value="25.0"/>
+<xacro:property name="wheel_mass" value="5.0"/>
+<xacro:property name="imu_width" value="0.036"/>
+<xacro:property name="imu_length" value="0.038"/>
+<xacro:property name="imu_height" value="0.012"/>
+<xacro:property name="imu_offset_x" value="0"/>
+<xacro:property name="imu_offset_y" value="0"/>
+<xacro:property name="imu_offset_z" value="${- body_height/2 + 0.005 + 0.007}"/>
+<xacro:property name="velodyne_height" value="0.1442"/>
+<xacro:property name="velodyne_radius" value="0.04265"/>
+<xacro:property name="velodyne_height_to_lense" value="0.090805"/>
+<xacro:property name="velodyne_offset_x" value="${body_length/2 - 0.0265 + 0.02}"/>
+<xacro:property name="velodyne_offset_y" value="0"/>
+<xacro:property name="velodyne_offset_z"
+  value="${0.2 + velodyne_height/2}"/>
+<link name="base_footprint" />
+<link name="base_link">
+    <visual>
+        <origin xyz="0 0 0" rpy="0 0 0" />
+        <geometry>
+            <box size="${body_length} ${body_width} ${body_height}"/>
+        </geometry>
+        <material name="silver" >
+            <color rgba="0.5 0.5 0.5 1" />
+        </material>
+    </visual>
+    <collision>
+        <origin xyz="0 0 0" rpy="0 0 0" />
+        <geometry>
+            <box size="${body_length} ${body_width} ${body_height}"/>
+        </geometry>
+    </collision>
+    <xacro:box_inertial
+        x="${body_length}"
+        y="${body_width}"
+        z="${body_height}"
+        mass="${body_mass}"/>
+</link>
+<joint name="base_footprint_to_base_joint" type="fixed">
+    <origin xyz="0 0 ${wheel_radius - axis_height}" rpy="0 0 0" />
+    <parent link="base_footprint" />
+    <child link="base_link" />
+</joint>
+<!--Wheel Macro-->
+<xacro:macro name="wheel" params="name parent xyz">
+  <link name="${name}_link">
+    <visual>
+      <origin xyz="0 0 0" rpy="${M_PI/2} 0 0" />
       <geometry>
-        <box size="${body_length} ${body_width} ${body_height}"/>
+        <cylinder length="${wheel_thickness}" radius="${wheel_radius}"/>
       </geometry>
-      <material name="silver" >
-        <color rgba="0.5 0.5 0.5 1" />
+      <material name="black" >
+        <color rgba="0 0 0 1" />
       </material>
     </visual>
     <collision>
-      <origin xyz="0 0 0" rpy="0 0 0" />
+      <origin xyz="0 0 0" rpy="${M_PI/2} 0 0" />
       <geometry>
-        <box size="${body_length} ${body_width} ${body_height}"/>
+        <cylinder length="${wheel_thickness}" radius="${wheel_radius}"/>
       </geometry>
     </collision>
-    <xacro:box_inertial
-      x="${body_length}"
-      y="${body_width}"
-      z="${body_height}"
-      mass="${body_mass}"/>
+    <xacro:cylinder_inertial_with_origin radius="${wheel_radius}" length="${wheel_thickness}" mass="${wheel_mass}">
+              <origin xyz="0 0 0" rpy="${M_PI/2} 0 0"/>
+    </xacro:cylinder_inertial_with_origin>
   </link>
-  <joint name="base_footprint_to_base_joint" type="fixed">
-    <origin xyz="0 0 ${wheel_radius - axis_height}" rpy="0 0 0" />
-    <parent link="base_footprint"/>
-    <child link="base_link" />
+  <joint name="${name}_joint" type="continuous">
+    <origin xyz="${xyz}" rpy="0 0 0"/>
+    <parent link="${parent}"/>
+    <child link="${name}_link"/>
+    <axis xyz="0 1 0"/>
   </joint>
-  <!--Wheel Macro-->
-  <xacro:macro name="wheel" params="name parent xyz">
-    <link name="${name}_link">
-      <visual>
-        <origin xyz="0 0 0" rpy="${M_PI/2} 0 0" />
+  <gazebo reference="${name}_link">
+    <mu1 value="0.7"/>
+    <mu2 value="0.7"/>
+    <kp value="100000000.0"/>
+    <kd value="10000.0"/>
+    <material>Gazebo/Black</material>
+    <selfCollide>false</selfCollide>
+  </gazebo>
+</xacro:macro>
+<xacro:macro name="box_for_joint" params="name o_x o_y o_z r_x r_y r_z r g b color length height width">
+  <link name="${name}_link">
+    <visual>
+      <origin xyz="${o_x} ${o_y} ${o_z}" rpy="${r_x} ${r_y} ${r_z}" />
+      <geometry>
+        <box size="${length} ${width} ${height}" />
+      </geometry>
+      <material name="${color}">
+        <color rgba="${r} ${g} ${b} 1"/>
+      </material>
+    </visual>
+  </link>
+</xacro:macro>
+<xacro:wheel
+  name="left_front_wheel"
+  parent="base_link"
+  xyz="${axis_front} ${axis_left} ${axis_height}" />
+<xacro:wheel
+  name="left_rear_wheel"
+  parent="base_link"
+  xyz="${axis_back} ${axis_left} ${axis_height}" />
+<xacro:wheel
+  name="right_front_wheel"
+  parent="base_link"
+  xyz="${axis_front} ${axis_right} ${axis_height}" />
+<xacro:wheel
+  name="right_rear_wheel"
+  parent="base_link"
+  xyz="${axis_back} ${axis_right} ${axis_height}" />
+<!-- Odom -->
+<gazebo>
+  <plugin name="skid_steer_drive_controller" filename="libgazebo_ros_skid_steer_drive.so">
+    <updateRate>100.0</updateRate>
+    <robotNamespace>/</robotNamespace>
+    <leftFrontJoint>left_front_wheel_joint</leftFrontJoint>
+    <rightFrontJoint>right_front_wheel_joint</rightFrontJoint>
+    <leftRearJoint>left_rear_wheel_joint</leftRearJoint>
+    <rightRearJoint>right_rear_wheel_joint</rightRearJoint>
+    <wheelSeparation>${axis_length}</wheelSeparation>
+    <wheelDiameter>${2*wheel_radius}</wheelDiameter>
+    <robotBaseFrame>base_link</robotBaseFrame>
+    <torque>30</torque>
+    <topicName>cmd_vel</topicName>
+    <broadcastTF>false</broadcastTF>
+  </plugin>
+</gazebo>
+<!-- IMU -->
+<link name="imu">
+    <visual>
+        <origin xyz="0 0 0" rpy="0 0 0" />
         <geometry>
-          <cylinder length="${wheel_thickness}" radius="${wheel_radius}"/>
+            <box size="${imu_length} ${imu_width} ${imu_height}"/>
         </geometry>
-        <material name="black" >
-          <color rgba="0 0 0 1" />
+        <material name="white" >
+            <color rgba="0.8 0.8 0.8 1" />
         </material>
-      </visual>
-      <collision>
-        <origin xyz="0 0 0" rpy="${M_PI/2} 0 0" />
-        <geometry>
-          <cylinder length="${wheel_thickness}" radius="${wheel_radius}"/>
-        </geometry>
-      </collision>
-      <xacro:cylinder_inertial
-        radius="${wheel_radius}"
-        length="${wheel_thickness}"
-        mass="${wheel_mass}" />
-    </link>
-    <joint name="${name}_joint" type="continuous">
-      <origin xyz="${xyz}" rpy="0 0 0"/>
-      <parent link="${parent}"/>
-      <child link="${name}_link"/>
-      <axis xyz="0 1 0"/>
-    </joint>
-    <gazebo reference="${name}_link">
-      <mu1 value="0.7"/>
-      <mu2 value="0.7"/>
-      <kp value="100000000.0"/>
-      <kd value="10000.0"/>
-      <material>Gazebo/Black</material>
-      <selfCollide>false</selfCollide>
-    </gazebo>
-  </xacro:macro>
-  <xacro:macro name="box_for_joint" params="name o_x o_y o_z r_x r_y r_z r g b color length height width">
-    <link name="${name}_link">
-      <visual>
-        <origin xyz="${o_x} ${o_y} ${o_z}" rpy="${r_x} ${r_y} ${r_z}" />
-        <geometry>
-          <box size="${length} ${width} ${height}" />
-        </geometry>
-        <material name="${color}">
-          <color rgba="${r} ${g} ${b} 1"/>
-        </material>
-      </visual>
-    </link>
-  </xacro:macro>
-  <xacro:wheel
-    name="left_front_wheel"
-    parent="base_link"
-    xyz="${axis_front} ${axis_left} ${axis_height}" />
-  <xacro:wheel
-    name="left_rear_wheel"
-    parent="base_link"
-    xyz="${axis_back} ${axis_left} ${axis_height}" />
-  <xacro:wheel
-    name="right_front_wheel"
-    parent="base_link"
-    xyz="${axis_front} ${axis_right} ${axis_height}" />
-  <xacro:wheel
-    name="right_rear_wheel"
-    parent="base_link"
-    xyz="${axis_back} ${axis_right} ${axis_height}" />
-  <link name="imu">
-    <visual>
-      <origin xyz="0 0 0" rpy="0 0 0" />
-      <geometry>
-        <box size="${imu_length} ${imu_width} ${imu_height}"/>
-      </geometry>
-      <material name="white" >
-        <color rgba="0.8 0.8 0.8 1" />
-      </material>
-    </visual>
-  </link>
-  <link name="em_body">
-    <visual>
-      <origin xyz="0 0 0" rpy="${M_PI/2} 0 ${M_PI/2}" />
-      <geometry>
-        <box size="${em_body_length} ${em_body_width} ${em_body_height}"/>
-      </geometry>
-      <material name="yellow">
-        <color rgba="1 1 0 1" />
-      </material>
-    </visual>
-  </link>
-  <link name="em_button">
-    <visual>
-      <origin xyz="0 0 0" rpy="0 ${M_PI/2} 0"/>
-      <geometry>
-        <cylinder length="${em_button_depth}" radius="${em_button_radius}"/>
-      </geometry>
-      <material name="red">
-        <color rgba="1 0 0 1"/>
-      </material>
-    </visual>
-  </link>
-  <joint name="em_body_to_base_joint" type="fixed">
-    <parent link="base_link" />
-    <child link="em_body" />
-    <origin
-      xyz=" ${-body_length/2}
-            0.03
-           -0.05
-          " />
-  </joint>
-  <joint name="em_button_to_em_body_joint" type="fixed">
-    <parent link="em_body" />
-    <child link="em_button" />
-    <origin
-      xyz=" ${-em_button_depth}
-            -0.02
-            0
-          " />
-  </joint>
-  <joint name="imu_to_base_joint" type="fixed">
+    </visual>
+</link>
+<!-- inertial measurement unit for gazebo -->
+<gazebo>
+    <plugin name="imu_controller" filename="libgazebo_ros_imu.so">
+    <alwaysOn>true</alwaysOn>
+    <updateRate>100.0</updateRate>
+    <bodyName>imu</bodyName>
+    <topicName>imu/data</topicName>
+    <serviceName>/default_imu</serviceName>
+    <gaussianNoise>${imu_stdev*imu_stdev}</gaussianNoise>
+    <xyzOffsets>0 0 0</xyzOffsets>
+    <rpyOffsets>0 0 0</rpyOffsets>
+    <interface:position name="imu_position"/>
+    </plugin>
+</gazebo>
+<joint name="imu_to_base_joint" type="fixed">
     <parent link="base_link" />
     <child link="imu" />
-    <origin
-      xyz=" ${imu_offset_x}
-            ${imu_offset_y}
-            ${imu_offset_z}"
-      rpy="${M_PI} 0 ${M_PI/2.0}" />
-  </joint>
-    <link name="velodyne">
-    <visual>
-      <origin xyz="0 0 ${-velodyne_height_to_lense}" rpy="0 0 0" />
-      <geometry>
-        <cylinder length="0.1442" radius="0.04265"/>
-      </geometry>
-      <material name="silver">
-        <color rgba="0.5 0.5 0.5 1" />
-      </material>
-    </visual>
-  </link>
-  <joint name="velodyne_to_base_joint" type="fixed">
-    <child link="velodyne" />
-    <parent link="base_link" />
-    <origin
-      xyz=" ${velodyne_offset_x}
-            ${velodyne_offset_y}
-            ${velodyne_offset_z + velodyne_height_to_lense}"
-      rpy="0 0 0" />
-  </joint>
-  <!-- inertial measurement unit for gazebo -->
-  <xacro:imu_gazebo link="imu" imu_topic="imu/data" update_rate="100.0" stdev="${imu_stdev}" />
-  <gazebo reference="velodyne">
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